Commit message: Stabilize robot simulation validation

File: src/robot_description/urdf/robot_base.urdf.xacro (robot description, xacro)
@@ -1,4 +1,4 @@
 <?xml version="1.0"?>
-<robot xmlns:xacro="http://www.ros.org/wiki/xacro" name="diff_drive_robot">
+<robot xmlns:xacro="http://www.ros.org/wiki/xacro" name="ackermann_robot">
   <!-- ==================== Constants ==================== -->
   <xacro:property name="PI" value="3.1415926535897931"/>
@@ -36,39 +36,222 @@
         <box size="${chassis_length} ${chassis_width} ${chassis_height}"/>
       </geometry>
-    </collision>
-  </link>
-  <!-- ==================== Wheels ==================== -->
-  <xacro:macro name="wheel" params="name x y">
-    <joint name="${name}_joint" type="continuous">
-      <parent link="base_link"/>
-      <child link="${name}_link"/>
-      <origin xyz="${x * wheelbase/2} ${y * track_width/2} ${-wheel_radius}" rpy="${PI/2} 0 0"/>
-      <axis xyz="0 0 1"/>
-      <dynamics damping="0.05" friction="0.1"/>
-    </joint>
-    <link name="${name}_link">
-      <inertial>
-        <mass value="0.5"/>
-        <inertia ixx="0.0002" ixy="0" ixz="0" iyy="0.0002" iyz="0" izz="0.0002"/>
-      </inertial>
-      <visual name="${name}_visual">
-        <geometry>
-          <cylinder radius="${wheel_radius}" length="${wheel_width}"/>
-        </geometry>
-        <material name="black">
-          <color rgba="0.1 0.1 0.1 1.0"/>
-        </material>
-      </visual>
-      <collision name="${name}_collision">
-        <geometry>
-          <cylinder radius="${wheel_radius}" length="${wheel_width}"/>
-        </geometry>
-      </collision>
-    </link>
-  </xacro:macro>
-  <xacro:wheel name="front_left" x="1" y="1"/>
-  <xacro:wheel name="front_right" x="1" y="-1"/>
-  <xacro:wheel name="rear_left" x="-1" y="1"/>
-  <xacro:wheel name="rear_right" x="-1" y="-1"/>
+      <surface>
+        <friction>
+          <ode>
+            <mu>0.8</mu>
+            <mu2>0.8</mu2>
+          </ode>
+        </friction>
+      </surface>
+    </collision>
+  </link>
+  <!-- ==================== Front Steering Joints ==================== -->
+  <joint name="left_steering_joint" type="fixed">
+    <parent link="base_link"/>
+    <child link="left_steering_link"/>
+    <origin xyz="${wheelbase/2} ${track_width/2} 0" rpy="0 0 0"/>
+  </joint>
+  <link name="left_steering_link">
+    <inertial>
+      <mass value="0.01"/>
+      <inertia ixx="0.001" ixy="0" ixz="0" iyy="0.001" iyz="0" izz="0.001"/>
+    </inertial>
+  </link>
+  <joint name="right_steering_joint" type="fixed">
+    <parent link="base_link"/>
+    <child link="right_steering_link"/>
+    <origin xyz="${wheelbase/2} ${-track_width/2} 0" rpy="0 0 0"/>
+  </joint>
+  <link name="right_steering_link">
+    <inertial>
+      <mass value="0.01"/>
+      <inertia ixx="0.001" ixy="0" ixz="0" iyy="0.001" iyz="0" izz="0.001"/>
+    </inertial>
+  </link>
+  <joint name="steering_wheel_joint" type="continuous">
+    <parent link="base_link"/>
+    <child link="steering_wheel_link"/>
+    <origin xyz="0.12 0 0.12" rpy="0 0 0"/>
+    <axis xyz="0 0 1"/>
+    <dynamics damping="0.1" friction="0.1"/>
+  </joint>
+  <link name="steering_wheel_link">
+    <inertial>
+      <mass value="0.01"/>
+      <inertia ixx="0.0001" ixy="0" ixz="0" iyy="0.0001" iyz="0" izz="0.0001"/>
+    </inertial>
+  </link>
+  <!-- ==================== Rear Fixed Joints ==================== -->
+  <joint name="rear_left_fixed_joint" type="fixed">
+    <parent link="base_link"/>
+    <child link="rear_left_fixed_link"/>
+    <origin xyz="${-wheelbase/2} ${track_width/2} 0" rpy="0 0 0"/>
+  </joint>
+  <link name="rear_left_fixed_link">
+    <inertial>
+      <mass value="0.01"/>
+      <inertia ixx="0.001" ixy="0" ixz="0" iyy="0.001" iyz="0" izz="0.001"/>
+    </inertial>
+  </link>
+  <joint name="rear_right_fixed_joint" type="fixed">
+    <parent link="base_link"/>
+    <child link="rear_right_fixed_link"/>
+    <origin xyz="${-wheelbase/2} ${-track_width/2} 0" rpy="0 0 0"/>
+  </joint>
+  <link name="rear_right_fixed_link">
+    <inertial>
+      <mass value="0.01"/>
+      <inertia ixx="0.001" ixy="0" ixz="0" iyy="0.001" iyz="0" izz="0.001"/>
+    </inertial>
+  </link>
+  <!-- ==================== Wheels (with proper rotation to stand upright) ==================== -->
+  <!-- Front Left Wheel -->
+  <joint name="front_left_joint" type="continuous">
+    <parent link="left_steering_link"/>
+    <child link="front_left_wheel"/>
+    <origin xyz="0 0 ${-wheel_radius + 0.02}" rpy="0 0 0"/>
+    <axis xyz="0 1 0"/>
+    <dynamics damping="0.05" friction="5.0"/>
+  </joint>
+  <link name="front_left_wheel">
+    <inertial>
+      <mass value="0.5"/>
+      <inertia ixx="0.0002" ixy="0" ixz="0" iyy="0.0002" iyz="0" izz="0.0002"/>
+    </inertial>
+    <visual name="front_left_wheel_visual">
+      <origin xyz="0 0 0" rpy="${PI/2} 0 0"/>
+      <geometry>
+        <cylinder radius="${wheel_radius}" length="${wheel_width}"/>
+      </geometry>
+      <material name="black">
+        <color rgba="0.1 0.1 0.1 1.0"/>
+      </material>
+    </visual>
+    <collision name="front_left_wheel_collision">
+      <origin xyz="0 0 0" rpy="${PI/2} 0 0"/>
+      <geometry>
+        <cylinder radius="${wheel_radius}" length="${wheel_width}"/>
+      </geometry>
+      <surface>
+        <friction>
+          <ode>
+            <mu>2.0</mu>
+            <mu2>2.0</mu2>
+          </ode>
+        </friction>
+      </surface>
+    </collision>
+  </link>
+  <!-- Front Right Wheel -->
+  <joint name="front_right_joint" type="continuous">
+    <parent link="right_steering_link"/>
+    <child link="front_right_wheel"/>
+    <origin xyz="0 0 ${-wheel_radius + 0.02}" rpy="0 0 0"/>
+    <axis xyz="0 1 0"/>
+    <dynamics damping="0.05" friction="5.0"/>
+  </joint>
+  <link name="front_right_wheel">
+    <inertial>
+      <mass value="0.5"/>
+      <inertia ixx="0.0002" ixy="0" ixz="0" iyy="0.0002" iyz="0" izz="0.0002"/>
+    </inertial>
+    <visual name="front_right_wheel_visual">
+      <origin xyz="0 0 0" rpy="${PI/2} 0 0"/>
+      <geometry>
+        <cylinder radius="${wheel_radius}" length="${wheel_width}"/>
+      </geometry>
+      <material name="black">
+        <color rgba="0.1 0.1 0.1 1.0"/>
+      </material>
+    </visual>
+    <collision name="front_right_wheel_collision">
+      <origin xyz="0 0 0" rpy="${PI/2} 0 0"/>
+      <geometry>
+        <cylinder radius="${wheel_radius}" length="${wheel_width}"/>
+      </geometry>
+      <surface>
+        <friction>
+          <ode>
+            <mu>2.0</mu>
+            <mu2>2.0</mu2>
+          </ode>
+        </friction>
+      </surface>
+    </collision>
+  </link>
+  <!-- Rear Left Wheel -->
+  <joint name="rear_left_joint" type="continuous">
+    <parent link="rear_left_fixed_link"/>
+    <child link="rear_left_wheel"/>
+    <origin xyz="0 0 ${-wheel_radius + 0.02}" rpy="0 0 0"/>
+    <axis xyz="0 1 0"/>
+    <dynamics damping="0.05" friction="5.0"/>
+  </joint>
+  <link name="rear_left_wheel">
+    <inertial>
+      <mass value="0.5"/>
+      <inertia ixx="0.0002" ixy="0" ixz="0" iyy="0.0002" iyz="0" izz="0.0002"/>
+    </inertial>
+    <visual name="rear_left_wheel_visual">
+      <origin xyz="0 0 0" rpy="${PI/2} 0 0"/>
+      <geometry>
+        <cylinder radius="${wheel_radius}" length="${wheel_width}"/>
+      </geometry>
+      <material name="black">
+        <color rgba="0.1 0.1 0.1 1.0"/>
+      </material>
+    </visual>
+    <collision name="rear_left_wheel_collision">
+      <origin xyz="0 0 0" rpy="${PI/2} 0 0"/>
+      <geometry>
+        <cylinder radius="${wheel_radius}" length="${wheel_width}"/>
+      </geometry>
+      <surface>
+        <friction>
+          <ode>
+            <mu>2.0</mu>
+            <mu2>2.0</mu2>
+          </ode>
+        </friction>
+      </surface>
+    </collision>
+  </link>
+  <!-- Rear Right Wheel -->
+  <joint name="rear_right_joint" type="continuous">
+    <parent link="rear_right_fixed_link"/>
+    <child link="rear_right_wheel"/>
+    <origin xyz="0 0 ${-wheel_radius + 0.02}" rpy="0 0 0"/>
+    <axis xyz="0 1 0"/>
+    <dynamics damping="0.05" friction="5.0"/>
+  </joint>
+  <link name="rear_right_wheel">
+    <inertial>
+      <mass value="0.5"/>
+      <inertia ixx="0.0002" ixy="0" ixz="0" iyy="0.0002" iyz="0" izz="0.0002"/>
+    </inertial>
+    <visual name="rear_right_wheel_visual">
+      <origin xyz="0 0 0" rpy="${PI/2} 0 0"/>
+      <geometry>
+        <cylinder radius="${wheel_radius}" length="${wheel_width}"/>
+      </geometry>
+      <material name="black">
+        <color rgba="0.1 0.1 0.1 1.0"/>
+      </material>
+    </visual>
+    <collision name="rear_right_wheel_collision">
+      <origin xyz="0 0 0" rpy="${PI/2} 0 0"/>
+      <geometry>
+        <cylinder radius="${wheel_radius}" length="${wheel_width}"/>
+      </geometry>
+      <surface>
+        <friction>
+          <ode>
+            <mu>2.0</mu>
+            <mu2>2.0</mu2>
+          </ode>
+        </friction>
+      </surface>
+    </collision>
+  </link>
   <!-- ==================== Sensor Links ==================== -->
   <joint name="imu_joint" type="fixed">
@@ -81,5 +264,5 @@
     <parent link="base_link"/>
     <child link="laser_link"/>
-    <origin xyz="0 0 ${lidar_height}" rpy="0 0 0"/>
+    <origin xyz="0 0 ${lidar_height}" rpy="0 0.524 0"/>
   </joint>
   <link name="laser_link">
@@ -89,4 +272,5 @@
     </inertial>
     <visual name="laser_visual">
+      <pose>0 0 0 0 1.5708 0</pose>
       <geometry>
         <cylinder radius="0.025" length="0.04"/>
@@ -97,4 +281,5 @@
     </visual>
     <collision name="laser_collision">
+      <pose>0 0 0 0 1.5708 0</pose>
       <geometry>
         <cylinder radius="0.025" length="0.04"/>
@@ -111,13 +296,17 @@
   <gazebo reference="imu_link">
     <sensor type="imu" name="imu_sensor">
+      <always_on>1</always_on>
+      <update_rate>100</update_rate>
       <plugin name="gazebo_ros_imu" filename="libgazebo_ros_imu_sensor.so">
-        <topicName>imu/data</topicName>
-        <bodyName>imu_link</bodyName>
-        <updateRateHZ>100</updateRateHZ>
+        <ros>
+          <namespace>/robot</namespace>
+          <remapping>~/out:=imu/data</remapping>
+        </ros>
+        <frame_name>imu_link</frame_name>
       </plugin>
     </sensor>
   </gazebo>
   <gazebo reference="laser_link">
-    <sensor type="ray" name="laser_sensor">
+    <sensor type="ray" name="velodyne_sensor">
       <always_on>1</always_on>
       <update_rate>10</update_rate>
@@ -130,18 +319,24 @@
             <max_angle>3.14159</max_angle>
           </horizontal>
+          <vertical>
+            <samples>16</samples>
+            <resolution>1</resolution>
+            <min_angle>-0.2618</min_angle>
+            <max_angle>0.2618</max_angle>
+          </vertical>
         </scan>
         <range>
           <min>0.1</min>
-          <max>30.0</max>
-          <resolution>0.02</resolution>
+          <max>100.0</max>
+          <resolution>0.01</resolution>
         </range>
       </ray>
-      <plugin name="gazebo_ros_laser" filename="libgazebo_ros_ray_sensor.so">
+      <plugin name="gazebo_ros_ray_sensor" filename="libgazebo_ros_ray_sensor.so">
         <ros>
           <namespace>/robot</namespace>
-          <remapping>~/out:=scan</remapping>
+          <remapping>~/out:=velodyne_points</remapping>
         </ros>
+        <output_type>sensor_msgs/PointCloud2</output_type>
         <frame_name>laser_link</frame_name>
-        <output_type>sensor_msgs/LaserScan</output_type>
       </plugin>
     </sensor>
@@ -149,10 +344,16 @@
   <gazebo reference="gps_link">
     <sensor type="gps" name="gps_sensor">
+      <always_on>1</always_on>
+      <update_rate>5</update_rate>
       <plugin name="gazebo_ros_gps" filename="libgazebo_ros_gps_sensor.so">
-        <topicName>gps/fix</topicName>
-        <frameName>gps_link</frameName>
+        <ros>
+          <namespace>/robot</namespace>
+          <remapping>~/out:=rtk_gps/fix</remapping>
+        </ros>
+        <frame_name>gps_link</frame_name>
       </plugin>
     </sensor>
   </gazebo>
+  <!-- ==================== Drive Plugin ==================== -->
   <gazebo>
     <plugin name="gazebo_ros_diff_drive" filename="libgazebo_ros_diff_drive.so">
@@ -160,14 +361,19 @@
         <namespace>/robot</namespace>
       </ros>
-      <update_rate>50</update_rate>
-      <left_joint>front_left_joint</left_joint>
-      <right_joint>front_right_joint</right_joint>
+      <update_rate>50.0</update_rate>
+      <left_joint>rear_left_joint</left_joint>
+      <right_joint>rear_right_joint</right_joint>
       <wheel_separation>${track_width}</wheel_separation>
       <wheel_diameter>${wheel_diameter}</wheel_diameter>
-      <max_wheel_torque>100</max_wheel_torque>
-      <max_wheel_acceleration>0.5</max_wheel_acceleration>
+      <max_wheel_torque>50</max_wheel_torque>
+      <max_wheel_acceleration>2.0</max_wheel_acceleration>
+      <command_topic>cmd_vel</command_topic>
+      <!-- Publishers -->
       <publish_odom>true</publish_odom>
       <publish_odom_tf>true</publish_odom_tf>
-      <publish_wheel_tf>true</publish_wheel_tf>
+      <publish_wheel_tf>false</publish_wheel_tf>
+      <odometry_topic>odom</odometry_topic>
+      <odometry_frame>odom</odometry_frame>
+      <robot_base_frame>base_footprint</robot_base_frame>
     </plugin>
   </gazebo>

Commit message: feat: ackermann drive controller, LIO-SAM2 localization, Nav2 integration

File: src/robot_description/urdf/robot_base.urdf.xacro (robot description, xacro)
@@ -47,8 +47,11 @@
   </link>
   <!-- ==================== Front Steering Joints ==================== -->
-  <joint name="left_steering_joint" type="fixed">
+  <joint name="left_steering_joint" type="revolute">
     <parent link="base_link"/>
     <child link="left_steering_link"/>
     <origin xyz="${wheelbase/2} ${track_width/2} 0" rpy="0 0 0"/>
+    <axis xyz="0 0 1"/>
+    <limit lower="-0.6" upper="0.6" effort="100" velocity="10"/>
+    <dynamics damping="0.1" friction="0.1"/>
   </joint>
   <link name="left_steering_link">
@@ -58,8 +61,11 @@
     </inertial>
   </link>
-  <joint name="right_steering_joint" type="fixed">
+  <joint name="right_steering_joint" type="revolute">
     <parent link="base_link"/>
     <child link="right_steering_link"/>
     <origin xyz="${wheelbase/2} ${-track_width/2} 0" rpy="0 0 0"/>
+    <axis xyz="0 0 1"/>
+    <limit lower="-0.6" upper="0.6" effort="100" velocity="10"/>
+    <dynamics damping="0.1" friction="0.1"/>
   </joint>
   <link name="right_steering_link">
@@ -112,5 +118,5 @@
     <origin xyz="0 0 ${-wheel_radius + 0.02}" rpy="0 0 0"/>
     <axis xyz="0 1 0"/>
-    <dynamics damping="0.05" friction="5.0"/>
+    <dynamics damping="0.01" friction="0.01"/>
   </joint>
   <link name="front_left_wheel">
@@ -149,5 +155,5 @@
     <origin xyz="0 0 ${-wheel_radius + 0.02}" rpy="0 0 0"/>
     <axis xyz="0 1 0"/>
-    <dynamics damping="0.05" friction="5.0"/>
+    <dynamics damping="0.01" friction="0.01"/>
   </joint>
   <link name="front_right_wheel">
@@ -186,5 +192,5 @@
     <origin xyz="0 0 ${-wheel_radius + 0.02}" rpy="0 0 0"/>
     <axis xyz="0 1 0"/>
-    <dynamics damping="0.05" friction="5.0"/>
+    <dynamics damping="0.01" friction="0.01"/>
   </joint>
   <link name="rear_left_wheel">
@@ -223,5 +229,5 @@
     <origin xyz="0 0 ${-wheel_radius + 0.02}" rpy="0 0 0"/>
     <axis xyz="0 1 0"/>
-    <dynamics damping="0.05" friction="5.0"/>
+    <dynamics damping="0.01" friction="0.01"/>
   </joint>
   <link name="rear_right_wheel">
@@ -355,25 +361,87 @@
     </sensor>
   </gazebo>
-  <!-- ==================== Drive Plugin ==================== -->
-  <gazebo>
-    <plugin name="gazebo_ros_diff_drive" filename="libgazebo_ros_diff_drive.so">
+  <!-- ==================== Ackermann Drive Controller ==================== -->
+  <gazebo>
+    <plugin name="ackermann_drive_controller" filename="libackermann_drive_controller.so">
       <ros>
         <namespace>/robot</namespace>
       </ros>
-      <update_rate>50.0</update_rate>
-      <left_joint>rear_left_joint</left_joint>
+      <cmd_vel_topic>cmd_vel</cmd_vel_topic>
+      <odom_topic>odom</odom_topic>
+      <ground_truth_odom_topic>ground_truth/odom</ground_truth_odom_topic>
+      <odom_frame>odom</odom_frame>
+      <base_frame>base_footprint</base_frame>
+      <left_steering_joint>left_steering_joint</left_steering_joint>
+      <right_steering_joint>right_steering_joint</right_steering_joint>
+      <rear_left_wheel_joint>rear_left_joint</rear_left_wheel_joint>
+      <rear_right_wheel_joint>rear_right_joint</rear_right_wheel_joint>
+      <wheelbase>${wheelbase}</wheelbase>
+      <track_width>${track_width}</track_width>
+      <wheel_radius>${wheel_radius}</wheel_radius>
+      <max_steering_angle>0.5236</max_steering_angle>
+      <cmd_timeout>0.5</cmd_timeout>
+      <update_rate>50.0</update_rate>
+      <steering_p>50.0</steering_p>
+      <steering_i>0.0</steering_i>
+      <steering_d>5.0</steering_d>
+      <max_wheel_torque>50.0</max_wheel_torque>
+    </plugin>
+  </gazebo>
+  <!-- ==================== Joint State Publisher ==================== -->
+  <gazebo>
+    <plugin name="gazebo_ros_joint_state_publisher" filename="libgazebo_ros_joint_state_publisher.so">
+      <ros>
+        <remapping>joint_states:=/joint_states</remapping>
+      </ros>
+      <update_rate>50.0</update_rate>
+      <joint_name>left_steering_joint</joint_name>
+      <joint_name>right_steering_joint</joint_name>
+      <joint_name>steering_wheel_joint</joint_name>
+      <joint_name>front_left_joint</joint_name>
+      <joint_name>front_right_joint</joint_name>
+      <joint_name>rear_left_joint</joint_name>
+      <joint_name>rear_right_joint</joint_name>
+    </plugin>
+  </gazebo>
+  <gazebo>
+    <plugin name="wheel_encoder_front_left" filename="libwheel_encoder.so">
+      <joint>front_left_joint</joint>
+      <topic>/robot/wheel_encoder/front_left</topic>
+      <update_rate>50.0</update_rate>
+      <output_type>angular_velocity</output_type>
+    </plugin>
+  </gazebo>
+  <gazebo>
+    <plugin name="wheel_encoder_front_right" filename="libwheel_encoder.so">
+      <joint>front_right_joint</joint>
+      <topic>/robot/wheel_encoder/front_right</topic>
+      <update_rate>50.0</update_rate>
+      <output_type>angular_velocity</output_type>
+    </plugin>
+  </gazebo>
+  <gazebo>
+    <plugin name="wheel_encoder_rear_left" filename="libwheel_encoder.so">
+      <joint>rear_left_joint</joint>
+      <topic>/robot/wheel_encoder/rear_left</topic>
+      <update_rate>50.0</update_rate>
+      <output_type>angular_velocity</output_type>
+    </plugin>
+  </gazebo>
+  <gazebo>
+    <plugin name="wheel_encoder_rear_right" filename="libwheel_encoder.so">
+      <joint>rear_right_joint</joint>
+      <topic>/robot/wheel_encoder/rear_right</topic>
+      <update_rate>50.0</update_rate>
+      <output_type>angular_velocity</output_type>
+    </plugin>
+  </gazebo>
+  <gazebo>
+    <plugin name="wheel_encoder_rear_average" filename="libwheel_encoder.so">
+      <joint>rear_left_joint</joint>
       <right_joint>rear_right_joint</right_joint>
-      <wheel_separation>${track_width}</wheel_separation>
-      <wheel_diameter>${wheel_diameter}</wheel_diameter>
-      <max_wheel_torque>50</max_wheel_torque>
-      <max_wheel_acceleration>2.0</max_wheel_acceleration>
-      <command_topic>cmd_vel</command_topic>
-      <!-- Publishers -->
-      <publish_odom>true</publish_odom>
-      <publish_odom_tf>true</publish_odom_tf>
-      <publish_wheel_tf>false</publish_wheel_tf>
-      <odometry_topic>odom</odometry_topic>
-      <odometry_frame>odom</odometry_frame>
-      <robot_base_frame>base_footprint</robot_base_frame>
+      <topic>/robot/wheel_encoder/rear_average</topic>
+      <update_rate>50.0</update_rate>
+      <wheel_radius>${wheel_radius}</wheel_radius>
+      <output_type>linear_velocity</output_type>
     </plugin>
   </gazebo>

Commit message: docs: 更新仿真导航交接与使用说明

File: src/robot_description/urdf/robot_base.urdf.xacro (robot description, xacro)
@@ -270,5 +270,5 @@
     <parent link="base_link"/>
     <child link="laser_link"/>
-    <origin xyz="0 0 ${lidar_height}" rpy="0 0.524 0"/>
+    <origin xyz="0 0 ${lidar_height}" rpy="0 0 0"/>
   </joint>
   <link name="laser_link">
